File: MCU datalogger.kicad_pcb (KiCad board)
At the start: 2 copper layers, 50.8 x 30.5 mm, 29 parts, among them J1 Conn_01x04_Pin, J2 Conn_01x04_Pin, J3 Conn_01x09_Pin, J4 Conn_02x03_Odd_Even, U1 24LC1025, U2 24LC1025, U3 ATMEGA328P-AU, U4 DS1337S_, Y1 32.768 KHz, Y2 16MHz

Commit message: added kicad logo
Parts:
- added REF**: KiCad-Logo2_5mm_SilkScreen, Symbol:KiCad-Logo2_5mm_SilkScreen, B.Cu at (121.3, 77.7)
